Commit message: add group state 'open' and 'close' for gripper

File: config/panda_arm_hand.srdf.xacro (robot description, xacro)
@@ -28,4 +28,12 @@
     <joint name="panda_joint7" value="0.785" />
   </group_state>
+  <group_state name="open" group="hand">
+    <joint name="panda_finger_joint1" value="0.035" />
+    <joint name="panda_finger_joint2" value="0.035" />
+  </group_state>
+  <group_state name="close" group="hand">
+    <joint name="panda_finger_joint1" value="0" />
+    <joint name="panda_finger_joint2" value="0" />
+    </group_state>
   <!--END EFFECTOR: Purpose: Represent information about an end effector.-->
   <end_effector name="hand" parent_link="panda_link8" group="hand" parent_group="panda_arm_hand" />

Commit message: Init

File: config/panda_arm_hand.srdf.xacro (robot description, xacro)
@@ -5,8 +5,12 @@
 -->
 <robot xmlns:xacro="http://www.ros.org/wiki/xacro" name="panda">
+  <!-- Initialize gripper_center properties -->
+  <xacro:arg name="gripper_center" default="false" />
+  <xacro:property name="gripper_center" value="$(arg gripper_center)"/>
+  <!-- Include other subgroup xacros -->
   <xacro:include filename="$(find panda_moveit_config)/config/panda_arm.xacro" />
   <xacro:include filename="$(find panda_moveit_config)/config/hand.xacro" />
   <xacro:panda_arm />
-  <xacro:hand />
+  <xacro:hand gripper_center="${gripper_center}"/>
   <!--GROUPS: Representation of a set of joints and links. This can be useful for specifying DOF to plan for, defining arms, end effectors, etc-->
   <!--LINKS: When a link is specified, the parent joint of that link (if it exists) is automatically included-->
@@ -37,5 +41,8 @@
     </group_state>
   <!--END EFFECTOR: Purpose: Represent information about an end effector.-->
-  <end_effector name="hand" parent_link="panda_link8" group="hand" parent_group="panda_arm_hand" />
+  <end_effector name="hand" parent_link="panda_link8" group="hand" parent_group="panda_arm" />
+  <xacro:if value="${gripper_center}"> <!-- Only when gripper_center==True -->
+    <end_effector name="gripper_center" parent_link="panda_gripper_center" group="panda_arm" parent_group="hand" />
+  </xacro:if>
   <!--DISABLE COLLISIONS: By default it is assumed that any link of the robot could potentially come into collision with any other link in the robot. This tag disables collision checking between a specified pair of links. -->
   <disable_collisions link1="panda_hand" link2="panda_link3" reason="Never" />
